File: KiCad/ardWaveFormGenerator/ardWaveformGenerator.kicad_sch (KiCad schematic)
At the start: 26 parts

Commit message: ardWaveformGenerator-0.2
Parts:
- removed C1, C2, C3, C4, C7, C8: (no value), symbol Device:CP
- removed RV1, RV2: (no value), symbol Device:R_POT
- added C1, C2, C3, C4, C7, C8: 1000u, My_Misc:CP_Radial_D10.0mm_P5.00mm_larger, symbol Device:C_Polarized
- added H1, H2, H3, H4: MountingHole, MountingHole:MountingHole_3.2mm_M3, symbol Mechanical:MountingHole
- added RV1: 10k, My_Headers:3-pin JST Potentiometer, symbol Device:R_Potentiometer
- added RV2: 50k, My_Headers:3-pin JST Potentiometer, symbol Device:R_Potentiometer
- A1: value (none) -> Arduino_Nano_v3.x; footprint (none) -> My_Arduino:Arduino_Nano_WithMountingHoles_larger
- C5, C6, C9: value (none) -> 100n; footprint (none) -> My_Misc:C_Rect_L7.0mm_W3.5mm_P5.00mm_larger
- D1: value (none) -> B40C2300-1500A; footprint (none) -> My_Misc:GBU-806
- F1: value (none) -> Fuse
- F2: value (none) -> Fuse; footprint (none) -> My_Headers:2-pin_Fuse_header_large
- J1: value (none) -> Conn_Coaxial; footprint (none) -> My_Headers:2-pin_Output_header_large
- J2: value (none) -> 4-pin_I2C_LCD_header; footprint (none) -> My_Headers:4-pin JST LCD
- R1: value (none) -> 2.2k; footprint (none) -> My_Misc:R_Axial_DIN0207_L6.3mm_D2.5mm_P10.16mm_Horizontal_large
- T1: value (none) -> Transformer_1P_SS
- U1: value (none) -> KY-040_Rotary_Encoder; footprint (none) -> My_Headers:5-pin JST Rotary Encoder
- U2: value (none) -> GY-9833_AD9833; footprint (none) -> My_Parts:GY-9833_AD9833_w_header_large
- U3: value (none) -> 3-pole_Power_input_screw_terminal; footprint (none) -> My_Parts:3-pole_screw_terminal_+12V,-12V_input
- U4: value (none) -> TL071; footprint (none) -> My_Misc:DIP-8_W7.62mm_large
- U5: value (none) -> LM7812_TO220; footprint (none) -> My_Parts:LM7812_TO-220-3_Vertical_larger
- U6: value (none) -> LM7912_TO220; footprint (none) -> My_Parts:LM7912_TO-220-3_Vertical_larger
- U7: value (none) -> LM7805_TO220; footprint (none) -> My_Parts:LM7805_TO-220-3_Vertical_larger
Connections:
- net +12V: now also C3.1, C7.1, RV1.1
- net +5V: now also C8.1
- net -12V: now also C4.2, RV1.3
- net GND: now also C1.2, C2.1, C3.2, C4.1, C7.2, C8.2
- net at D1.1 (-), U6.2 (VI): now also C2.2
- net at D1.4 (+), U5.1 (VI): now also C1.1
- net at R1.1, U4.2 (-): now also RV2.2
- net at J1.1 (In), U4.6: now also RV2.1
- net at U4.3 (+): now also RV1.2
Other:
- title: (none) -> ardWaveformGenerator
