File: KiCad/ardToneGenerator/ardToneGenerator.kicad_sch (KiCad schematic)
At the start: 36 parts

Commit message: ardToneGenerator-0.1
Parts:
- removed J1: (no value), symbol My_Headers:3-pin_LCD_header
- removed J? (x2): (no value), symbol My_Headers:2-pin_NO_switch_header
- added J1: Output, My_Headers:2-pin_Output_header_large, symbol My_Headers:2-pin_Audio
- added J2: 5-pin_LCD, My_Headers:5-pin JST LiquidCrystal595, symbol My_Headers:5-pin_LCD
- added J3: 3-pin_2-buttons, My_Headers:3-pin JST 2-buttons, symbol My_Headers:3-pin_2-buttons
- A1: value (none) -> Arduino_UNO_R3; footprint (none) -> My_Arduino:Arduino_UNO_R3_shield_large
- C1, C2: renamed from C?; value (none) -> 0.47u; footprint (none) -> My_Misc:C_Disc_D3.0mm_W1.6mm_P2.50mm_larg
- R1, R10, R11, R12, R13, R14, R15, R16, R17, R18, R19, R2, R20, R21, R22, R23, R24, R25, R26, R3, R4, R5, R6, R7, R8, R9: value (none) -> 10k; footprint (none) -> My_Misc:R_Axial_DIN0207_L6.3mm_D2.5mm_P10.16mm_Horizontal_large
- R27, R28, R29: renamed from R?; value (none) -> 10k; footprint (none) -> My_Misc:R_Axial_DIN0207_L6.3mm_D2.5mm_P10.16mm_Horizontal_large
- U1: renamed from U?; value (none) -> KY-040_Rotary_Encoder; footprint (none) -> My_Headers:5-pin JST Rotary Encoder
Connections:
- net Out- is gone; now on net GND: A1.29 (GND), R18.1
- net at A1.10 (A1), R28.1: now also J3.1 (+)
- net at A1.23 (D8): now also J2.1 (Data)
- net at A1.24 (D9): now also J2.2 (Latch)
- net at A1.25 (D10): now also J2.3 (Clock)
- net at A1.5 (+5V), R29.1, U1.4 (VCC): now also J3.3 (Sig)
- net GND: now reaches A1.6 (GND)
- net GND: now also A1.7 (GND), C1.2, C2.2, R27.2, R28.2, U1.5 (GND), J1.2 (-), J2.5 (GND)
- net at A1.9 (A0): now also R27.1, J3.2 (Sig)
- net Out+: no longer names the net of R17.2, R8.2
- net Out+: now also J1.1 (+)
- new net +5V: J2.4 (+5V)
Other:
- title: (none) -> ardToneGenerator
