File: KiCad/ardToneGeneratorJK/ardToneGeneratorJK.kicad_sch (KiCad schematic)
At the start: 31 parts

Commit message: ardWaveformGenerator-AG-pio with pcb-0.2
Parts:
- removed J1: (no value), symbol My_Headers:3-pin_LCD_header
- removed RV1, RV2, RV3: (no value), symbol Device:R_POT
- added J1: Output, My_Headers:2-pin_Output_header, symbol My_Headers:2-pin_Audio
- added J2: 5-pin_LCD, My_Headers:5-pin JST LCD, symbol My_Headers:5-pin_LCD
- added RV1, RV2, RV3: 10k, My_Headers:3-pin JST Potentiometer, symbol Device:R_Potentiometer
- A1: value (none) -> Arduino_UNO_R3; footprint (none) -> My_Arduino:Arduino_UNO_R3_shield_large
- R1, R10, R11, R12, R13, R14, R15, R16, R17, R18, R19, R2, R20, R21, R22, R23, R24, R25, R26, R3, R4, R5, R6, R7, R8, R9: value (none) -> 10k; footprint (none) -> My_Misc:R_Axial_DIN0207_L6.3mm_D2.5mm_P10.16mm_Horizontal_large
Connections:
- net at A1.10 (A1): now also RV2.2
- net at A1.11 (A2): now also RV3.2
- net at A1.23 (D8): now also J2.1 (Data)
- net at A1.24 (D9): now also J2.2 (Latch)
- net at A1.25 (D10): now also J2.3 (Clock)
- net at A1.5 (+5V): now also RV1.1, RV2.1, RV3.1
- net at A1.7 (GND): now also RV1.3, RV2.3, RV3.3
- net at A1.9 (A0): now also RV1.2
- net Out+: no longer names the net of R17.2, R8.2
- net Out+: now also J1.1 (+)
- net Out-: no longer names the net of A1.29 (GND), R18.1
- net Out-: now also J1.2 (-)
- new net +5V: J2.4 (+5V)
- new net GND: J2.5 (GND)
