File: KiCad/ardWaveformGenerator-AG/ArduinoUNO_sch.kicad_sch (KiCad schematic)
At the start: 1 part

Commit message: ardWaveformGenerator-AG-pio with pcb-0.2
Connections:
- net A4: no longer A1.31 (SDA/A4)
- net A5: no longer A1.32 (SCL/A5)
- net D0: no longer A1.27 (D12)
- new net D12: A1.27 (D12)
Changed lines of the file:
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@@
-    (stroke (width 0) (type default) (color 0 0 0 0))
-  )
-  (wire (pts (xy 166.37 110.49) (xy 181.61 110.49))
-    (stroke (width 0) (type default) (color 0 0 0 0))
-  )
-  (wire (pts (xy 166.37 107.95) (xy 171.45 107.95))
     (stroke (width 0) (type default) (color 0 0 0 0))
   )
@@
     )
   )
-  (global_label "D0" (shape input) (at 135.89 105.41 180) (fields_autoplaced)
+  (global_label "D12" (shape input) (at 135.89 105.41 180) (fields_autoplaced)
     (effects (font (size 1.27 1.27)) (justify right))
-    (property "Intersheet References" "${INTERSHEET_REFS}" (id 0) (at 130.9974 105.3306 0)
+    (property "Intersheet References" "${INTERSHEET_REFS}" (id 0) (at 129.7879 105.3306 0)
       (effects (font (size 1.27 1.27)) (justify right) hide)
     )
@@
     )
   )
-  (global_label "A5" (shape input) (at 181.61 110.49 0) (fields_autoplaced)
-    (effects (font (size 1.27 1.27)) (justify left))
-    (property "Intersheet References" "${INTERSHEET_REFS}" (id 0) (at 186.3212 110.4106 0)
-      (effects (font (size 1.27 1.27)) (justify left) hide)
-    )
-  )
   (global_label "D6" (shape input) (at 135.89 90.17 180) (fields_autoplaced)
     (effects (font (size 1.27 1.27)) (justify right))
@@
     )
   )
-  (global_label "A4" (shape input) (at 171.45 107.95 0) (fields_autoplaced)
-    (effects (font (size 1.27 1.27)) (justify left))
-    (property "Intersheet References" "${INTERSHEET_REFS}" (id 0) (at 176.1612 107.8706 0)
-      (effects (font (size 1.27 1.27)) (justify left) hide)
-    )
-  )
